File: ros2/main.kicad_pcb (KiCad board)
At the start: 2 copper layers, 9 parts, among them J1 Battery, U1 ESP32-DEVKIT-V1, U2 TB6612NFG, U3 TB6612NFG, U4 ACS712, U5 XL63070, U6 ZC323900, U7 TB6612NFG, U8 TB6612NFG

Commit message: schema without esp32
Parts:
- added J2: BMS_input, Connector_Wire:SolderWire-1sqmm_1x03_P5.4mm_D1.4mm_OD2.7mm, F.Cu at (65.2, 21.0)
- added J3: BMS_output, Connector_Wire:SolderWire-1sqmm_1x02_P5.4mm_D1.4mm_OD2.7mm, F.Cu at (118.6, 104.1)
- added J5: SWITCH_CONNECTOR, Connector_Wire:SolderWire-1sqmm_1x02_P5.4mm_D1.4mm_OD2.7mm, F.Cu at (178.4, 95.2)
- added J_M1_ENCODER1: Conn_01x04, Connector_PinHeader_2.54mm:PinHeader_1x04_P2.54mm_Vertical, F.Cu at (26.4, 141.6)
- added J_M1_POWER1: Conn_01x02, TerminalBlock:TerminalBlock_Xinya_XY308-2.54-2P_1x02_P2.54mm_Horizontal, F.Cu at (42.4, 36.9)
- added J_M2_ENCODER1: Conn_01x04, Connector_PinHeader_2.54mm:PinHeader_1x04_P2.54mm_Vertical, F.Cu at (151.5, 106.4)
- added J_M2_POWER1: Conn_01x02, TerminalBlock:TerminalBlock_Xinya_XY308-2.54-2P_1x02_P2.54mm_Horizontal, F.Cu at (34.8, 45.4)
- added J_M3_ENCODER1: Conn_01x04, Connector_PinHeader_2.54mm:PinHeader_1x04_P2.54mm_Vertical, F.Cu at (156.1, 106.4)
- added J_M3_POWER1: Conn_01x02, TerminalBlock:TerminalBlock_Xinya_XY308-2.54-2P_1x02_P2.54mm_Horizontal, F.Cu at (34.8, 53.0)
- added J_M4_ENCODER1: Conn_01x04, Connector_PinHeader_2.54mm:PinHeader_1x04_P2.54mm_Vertical, F.Cu at (160.2, 106.7)
- added J_M4_POWER1: Conn_01x02, TerminalBlock:TerminalBlock_Xinya_XY308-2.54-2P_1x02_P2.54mm_Horizontal, F.Cu at (65.3, 70.0)
- J1: value Battery -> Battery Conn_01x02; footprint Battery:Connector -> TerminalBlock:TerminalBlock_Xinya_XY308-2.54-2P_1x02_P2.54mm_Horizontal
- U4: value ACS712 -> TB6612NFG; footprint Package_SO:SOIC-8_3.9x4.9mm_P1.27mm -> tb6612fng:MODULE_ROB-14450
- U5: value XL63070 -> TB6612NFG; footprint XL63070:XL63070_Module_30x16 -> tb6612fng:MODULE_ROB-14450
- U6: value ZC323900 -> TXS0108E
- U7: value TB6612NFG -> ~; footprint tb6612fng:MODULE_ROB-14450 -> ACS712_MODULE:ACS712_module
- U8: value TB6612NFG -> XL63070; footprint tb6612fng:MODULE_ROB-14450 -> XL63070:XL63070_Module_30x16
- moved J1 190.5 mm to (47.7, 23.7), turned to -90 degrees
- moved U1 148.2 mm to (80.4, 110.8)
- moved U7 96.6 mm to (160.7, 79.5)
- moved U8 92.3 mm to (156.3, 156.9)
- moved U2 84.8 mm to (90.0, 41.4)
- moved U3 84.2 mm to (145.3, 40.0)
- moved U4 75.6 mm to (118.8, 72.2)
- moved U6 73.4 mm to (209.2, 146.9), turned to 0 degrees
- moved U5 45.1 mm to (190.6, 61.5), turned to 0 degrees
Connections:
- J1 pad 1: /POWER+ -> /BAT_RAW_PLUS
- J1 pad 2: /POWER- -> /BAT_RAW_MINUS
- U1 pad 30: unconnected-(U1-VIN-Pad30) -> +5V
- U2 pad 1: unconnected-(U2-VM-Pad1) -> /POWER+
- U2 pad 10: unconnected-(U2-PWMB-Pad10) -> /M2_PWM
- U2 pad 11: unconnected-(U2-BI2-Pad11) -> /M2_IN2
- U2 pad 12: unconnected-(U2-BI1-Pad12) -> /M2_IN1
- U2 pad 13: unconnected-(U2-STBY-Pad13) -> /MOTORS_STBY
- U2 pad 14: unconnected-(U2-AI1-Pad14) -> /M2_IN1
- U2 pad 15: unconnected-(U2-AI2-Pad15) -> /M2_IN2
- U2 pad 16: unconnected-(U2-PWMA-Pad16) -> /M2_PWM
- U2 pad 2: +5V -> +3.3V
- U2 pad 4: unconnected-(U2-A01-Pad4) -> /M2_OUT1
- U2 pad 5: unconnected-(U2-A02-Pad5) -> /M2_OUT2
- U2 pad 6: unconnected-(U2-B02-Pad6) -> /M2_OUT2
- U2 pad 7: unconnected-(U2-B01-Pad7) -> /M2_OUT1
- U3 pad 1: unconnected-(U3-VM-Pad1) -> /POWER+
- U3 pad 10: unconnected-(U3-PWMB-Pad10) -> /M3_PWM
- U3 pad 11: unconnected-(U3-BI2-Pad11) -> /M3_IN2
- U3 pad 12: unconnected-(U3-BI1-Pad12) -> /M3_IN1
- U3 pad 13: unconnected-(U3-STBY-Pad13) -> /MOTORS_STBY
- U3 pad 14: unconnected-(U3-AI1-Pad14) -> /M3_IN1
- U3 pad 15: unconnected-(U3-AI2-Pad15) -> /M3_IN2
- U3 pad 16: unconnected-(U3-PWMA-Pad16) -> /M3_PWM
- U3 pad 2: +5V -> +3.3V
- U3 pad 4: unconnected-(U3-A01-Pad4) -> /M3_OUT1
- U3 pad 5: unconnected-(U3-A02-Pad5) -> /M3_OUT2
- U3 pad 6: unconnected-(U3-B02-Pad6) -> /M3_OUT2
- U3 pad 7: unconnected-(U3-B01-Pad7) -> /M3_OUT1
- U4 pad 2: /POWER+ -> +3.3V
- U4 pad 3: /POWER- -> GNDD
- U4 pad 4: /POWER- -> /M4_OUT1
- U4 pad 5: GNDD -> /M4_OUT2
- U4 pad 6: Net-(U4-FILTR) -> /M4_OUT2
- U4 pad 7: unconnected-(U4-VIOUT-Pad7) -> /M4_OUT1
- U4 pad 8: +5V -> GNDD
- U5 pad 2: /POWER- -> +3.3V
- U5 pad 4: +5V -> /M1_OUT1
- U6 pad 1: unconnected-(U6-VA-Pad1) -> +3.3V
- U6 pad 10: unconnected-(U6-OE-Pad10) -> /TXS_OE
- U6 pad 12: unconnected-(U6-B8-Pad12) -> /M4_ENC_B
- U6 pad 13: unconnected-(U6-B7-Pad13) -> /M4_ENC_A
- U6 pad 14: unconnected-(U6-B6-Pad14) -> /M3_ENC_B
- U6 pad 15: unconnected-(U6-B5-Pad15) -> /M3_ENC_A
- U6 pad 16: unconnected-(U6-B4-Pad16) -> /M2_ENC_B
- U6 pad 17: unconnected-(U6-B3-Pad17) -> /M2_ENC_A
- U6 pad 18: unconnected-(U6-B2-Pad18) -> /M1_ENC_B
- U6 pad 19: unconnected-(U6-B1-Pad19) -> /M1_ENC_A
- U6 pad 2: unconnected-(U6-A1-Pad2) -> /M1_ENC_A_ESP
- U6 pad 20: unconnected-(U6-VB-Pad20) -> +5V
- U6 pad 3: unconnected-(U6-A2-Pad3) -> /M1_ENC_B_ESP
- U6 pad 4: unconnected-(U6-A3-Pad4) -> /M2_ENC_A_ESP
- U6 pad 5: unconnected-(U6-A4-Pad5) -> /M2_ENC_B_ESP
- U6 pad 6: unconnected-(U6-A5-Pad6) -> /M3_ENC_A_ESP
- U6 pad 7: unconnected-(U6-A6-Pad7) -> /M3_ENC_B_ESP
- U6 pad 8: unconnected-(U6-A7-Pad8) -> /M4_ENC_A_ESP
- U6 pad 9: unconnected-(U6-A8-Pad9) -> /M4_ENC_B_ESP
- U7 pad 1: unconnected-(U7-VM-Pad1) -> +5V
- U7 pad 2: +5V -> Net-(U7-OUT)
- U8 pad 1: unconnected-(U8-VM-Pad1) -> /POWER+
- U8 pad 2: +5V -> GNDD
- U8 pad 4: unconnected-(U8-A01-Pad4) -> +5V

Commit message: add esp32 connections
Parts:
- added C1: 100nF, Capacitor_THT:C_Disc_D5.0mm_W2.5mm_P5.00mm, F.Cu at (250.4, 31.9)
- added C10: 220uF, Capacitor_THT:CP_Radial_D10.0mm_P3.50mm, F.Cu at (233.3, 70.3)
- added C13: 100nF, Capacitor_THT:C_Disc_D5.0mm_W2.5mm_P5.00mm, F.Cu at (250.4, 56.2)
- added C14: 10uF, Capacitor_THT:C_Disc_D5.0mm_W2.5mm_P5.00mm, F.Cu at (258.5, 31.9)
- added C15: 22uF, Capacitor_THT:C_Disc_D5.0mm_W2.5mm_P5.00mm, F.Cu at (258.5, 36.0)
- added C16: 100nF, Capacitor_THT:C_Disc_D5.0mm_W2.5mm_P5.00mm, F.Cu at (258.5, 40.0)
- added C17: 2200uF, Capacitor_THT:CP_Radial_D12.5mm_P5.00mm, F.Cu at (253.7, 65.3)
- added C18: 100nF, Capacitor_THT:C_Disc_D5.0mm_W2.5mm_P5.00mm, F.Cu at (258.5, 44.1)
- added C19: 100nF, Capacitor_THT:C_Disc_D5.0mm_W2.5mm_P5.00mm, F.Cu at (258.5, 48.1)
- added C2: 10uF, Capacitor_THT:C_Disc_D5.0mm_W2.5mm_P5.00mm, F.Cu at (250.4, 36.0)
- added C20: 100nF, Capacitor_THT:C_Disc_D5.0mm_W2.5mm_P5.00mm, F.Cu at (258.5, 52.2)
- added C21: 100nF, Capacitor_THT:C_Disc_D5.0mm_W2.5mm_P5.00mm, F.Cu at (258.5, 56.2)
- added C3: 22nF, Capacitor_THT:C_Disc_D5.0mm_W2.5mm_P5.00mm, F.Cu at (250.4, 40.0)
- added C4: 220uF, Capacitor_THT:CP_Radial_D10.0mm_P3.50mm, F.Cu at (233.3, 35.7)
- added C5: 22nF, Capacitor_THT:C_Disc_D5.0mm_W2.5mm_P5.00mm, F.Cu at (250.4, 44.1)
- added C6: 220uF, Capacitor_THT:CP_Radial_D10.0mm_P3.50mm, F.Cu at (233.3, 47.2)
- added C7: 22nF, Capacitor_THT:C_Disc_D5.0mm_W2.5mm_P5.00mm, F.Cu at (250.4, 48.1)
- added C8: 220uF, Capacitor_THT:CP_Radial_D10.0mm_P3.50mm, F.Cu at (233.3, 58.8)
- added C9: 22nF, Capacitor_THT:C_Disc_D5.0mm_W2.5mm_P5.00mm, F.Cu at (250.4, 52.2)
- added D1: LED, LED_THT:LED_D5.0mm, F.Cu at (265.7, 62.0)
- added H1: MountingHole, MountingHole:MountingHole_3.2mm_M3, F.Cu at (244.8, 33.9)
- added H2: MountingHole, MountingHole:MountingHole_3.2mm_M3, F.Cu at (244.8, 41.8)
- added H3: MountingHole, MountingHole:MountingHole_3.2mm_M3, F.Cu at (244.8, 49.8)
- added H4: MountingHole, MountingHole:MountingHole_3.2mm_M3, F.Cu at (244.8, 57.7)
- added J6: ACS_IN, Connector_Wire:SolderWire-1sqmm_1x01_D1.4mm_OD2.7mm, F.Cu at (118.6, 154.5)
- added J7: ACS_POWER_OUT, Connector_Wire:SolderWire-1sqmm_1x01_D1.4mm_OD2.7mm, F.Cu at (118.6, 159.3)
- added R1: 1k, Resistor_THT:R_Axial_DIN0207_L6.3mm_D2.5mm_P7.62mm_Horizontal, F.Cu at (266.7, 31.9)
- added R2: 10К, Resistor_THT:R_Axial_DIN0207_L6.3mm_D2.5mm_P7.62mm_Horizontal, F.Cu at (266.7, 36.0)
- added R3: 100K, Resistor_THT:R_Axial_DIN0207_L6.3mm_D2.5mm_P7.62mm_Horizontal, F.Cu at (266.7, 40.0)
- added R4: 10K, Resistor_THT:R_Axial_DIN0207_L6.3mm_D2.5mm_P7.62mm_Horizontal, F.Cu at (266.7, 44.1)
- added R5: 30К, Resistor_THT:R_Axial_DIN0207_L6.3mm_D2.5mm_P7.62mm_Horizontal, F.Cu at (266.7, 48.1)
- added R6: 10K, Resistor_THT:R_Axial_DIN0207_L6.3mm_D2.5mm_P7.62mm_Horizontal, F.Cu at (266.7, 52.2)
- J5: value SWITCH_CONNECTOR -> SW_CONNECTOR
- U7: value ~ -> ACS712_MODULE
- moved U6 24.1 mm to (221.5, 126.2), turned to 180 degrees
- moved J_M3_POWER1 7.28 mm to (32.2, 59.9)
Connections:
- J5 pad 2: /POWER+ -> /SWITCHED_PLUS
- U1 pad 10: unconnected-(U1-D19-Pad10) -> /M2_PWM
- U1 pad 11: unconnected-(U1-D21-Pad11) -> /M3_PWM
- U1 pad 14: unconnected-(U1-D22-Pad14) -> /M4_PWM
- U1 pad 15: unconnected-(U1-D23-Pad15) -> /LEFT_IN1
- U1 pad 17: unconnected-(U1-VP-Pad17) -> /VBAT_ADC
- U1 pad 18: unconnected-(U1-VN-Pad18) -> /ACS_ESP
- U1 pad 19: unconnected-(U1-D34-Pad19) -> /M1_ENC_A_ESP
- U1 pad 20: unconnected-(U1-D35-Pad20) -> /M1_ENC_B_ESP
- U1 pad 21: unconnected-(U1-D32-Pad21) -> /M2_ENC_A_ESP
- U1 pad 22: unconnected-(U1-D33-Pad22) -> /M2_ENC_B_ESP
- U1 pad 23: unconnected-(U1-D25-Pad23) -> /LEFT_IN2
- U1 pad 24: unconnected-(U1-D26-Pad24) -> /RIGHT_IN1
- U1 pad 25: unconnected-(U1-D27-Pad25) -> /RIGHT_IN2
- U1 pad 26: unconnected-(U1-D14-Pad26) -> /M3_ENC_A_ESP
- U1 pad 28: unconnected-(U1-D13-Pad28) -> /MOTORS_STBY
- U1 pad 4: unconnected-(U1-D2-Pad4) -> /TXS_OE
- U1 pad 5: unconnected-(U1-D4-Pad5) -> /M4_ENC_B_ESP
- U1 pad 6: unconnected-(U1-RX2-Pad6) -> /M3_ENC_B_ESP
- U1 pad 7: unconnected-(U1-TX2-Pad7) -> /M4_ENC_A_ESP
- U1 pad 9: unconnected-(U1-D18-Pad9) -> /M1_PWM
- U2 pad 11: /M2_IN2 -> /LEFT_IN2
- U2 pad 12: /M2_IN1 -> /LEFT_IN1
- U2 pad 14: /M2_IN1 -> /LEFT_IN1
- U2 pad 15: /M2_IN2 -> /LEFT_IN2
- U3 pad 11: /M3_IN2 -> /RIGHT_IN2
- U3 pad 12: /M3_IN1 -> /RIGHT_IN1
- U3 pad 14: /M3_IN1 -> /RIGHT_IN1
- U3 pad 15: /M3_IN2 -> /RIGHT_IN2
- U4 pad 11: /M4_IN2 -> /RIGHT_IN2
- U4 pad 12: /M4_IN1 -> /RIGHT_IN1
- U4 pad 14: /M4_IN1 -> /RIGHT_IN1
- U4 pad 15: /M4_IN2 -> /RIGHT_IN2
- U5 pad 11: /M1_IN2 -> /LEFT_IN2
- U5 pad 12: /M1_IN1 -> /LEFT_IN1
- U5 pad 14: /M1_IN1 -> /LEFT_IN1
- U5 pad 15: /M1_IN2 -> /LEFT_IN2

Commit message: saved details
Parts:
- removed U1: ESP32-DEVKIT-V1, esp32:MODULE_ESP32_DEVKIT_V1
- U7: footprint ACS712_MODULE:ACS712_module -> Connector_PinSocket_2.54mm:PinSocket_1x03_P2.54mm_Vertical
- moved D1 138.4 mm to (133.4, 102.6)
- moved R1 137.6 mm to (140.4, 86.6)
- moved R2 137.6 mm to (140.4, 90.6)
- moved R3 137.6 mm to (140.4, 94.7)
- moved R4 137.6 mm to (140.4, 98.7)
- moved R5 137.6 mm to (140.4, 102.8)
- moved R6 137.6 mm to (140.4, 106.8)
- moved J_M1_ENCODER1 136.9 mm to (151.9, 86.9)
- moved J_M3_POWER1 124.2 mm to (156.4, 62.3), turned to 0 degrees
- moved J2 117.0 mm to (152.3, 99.2), turned to 0 degrees
- moved H1 116.0 mm to (134.9, 71.0)
- moved H2 116.0 mm to (134.9, 78.9)
- moved H3 116.0 mm to (134.9, 86.9)
- moved H4 116.0 mm to (134.9, 94.8)
- moved J_M2_POWER1 115.2 mm to (148.7, 62.3), turned to 0 degrees
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
Commit message: fix 2
Parts:
- added C11: 100nF, Capacitor_THT:C_Disc_D5.0mm_W2.5mm_P5.00mm, F.Cu at (203.1, 60.5)
- added C12: 10uF, Capacitor_THT:C_Disc_D5.0mm_W2.5mm_P5.00mm, F.Cu at (203.1, 64.5)
- D1: value LED -> LED_RED

Commit message: routed pcb + corrected schematic
Parts:
- removed J1: Battery Conn_01x02, TerminalBlock:TerminalBlock_Xinya_XY308-2.54-2P_1x02_P2.54mm_Horizontal
- added J4: Conn_01x03, Connector_Wire:SolderWire-1sqmm_1x03_P5.4mm_D1.4mm_OD2.7mm, F.Cu at (175.4, 128.0)
- added U1: ESP32-DEVKIT-V1, esp32:MODULE_ESP32_DEVKIT_V1, F.Cu at (152.3, 69.7)
- C3, C5, C7, C9: value 22nF -> 100nF
- U7: footprint Connector_PinSocket_2.54mm:PinSocket_1x03_P2.54mm_Vertical -> ACS712_MODULE:ACS712_module
- moved H4 95.8 mm to (199.1, 23.8)
- moved H2 84.0 mm to (199.2, 133.0)
- moved U5 71.8 mm to (125.8, 63.8)
- moved C18 68.8 mm to (142.7, 23.4)
- moved H3 68.2 mm to (109.0, 23.8)
- moved H1 67.2 mm to (109.0, 133.0)
- moved C15 66.5 mm to (124.5, 109.6), turned to -90 degrees
- moved C6 64.8 mm to (180.7, 105.7)
- moved U6 63.5 mm to (153.9, 32.9), turned to 90 degrees
- moved C9 62.9 mm to (121.4, 51.8)
- moved C16 61.7 mm to (127.7, 109.6), turned to -90 degrees
- moved R3 58.1 mm to (165.9, 42.5), turned to 180 degrees
- moved C19 56.9 mm to (142.6, 42.5), turned to 180 degrees
- moved C14 54.3 mm to (148.4, 113.1), turned to -90 degrees
- moved C8 51.9 mm to (172.3, 104.4), turned to 90 degrees
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Connections:
- J2 pad 3: /BAT_RAW_MINUS -> GNDD
- J_M1_ENCODER1 pad 2: GNDD -> /M1_ENC_A
- J_M1_ENCODER1 pad 3: /M1_ENC_A -> /M1_ENC_B
- J_M1_ENCODER1 pad 4: /M1_ENC_B -> GNDD
- J_M2_ENCODER1 pad 2: GNDD -> /M3_ENC_A
- J_M2_ENCODER1 pad 3: /M3_ENC_A -> /M3_ENC_B
- J_M2_ENCODER1 pad 4: /M3_ENC_B -> GNDD
- J_M3_ENCODER1 pad 2: GNDD -> /M2_ENC_A
- J_M3_ENCODER1 pad 3: /M2_ENC_A -> /M2_ENC_B
- J_M3_ENCODER1 pad 4: /M2_ENC_B -> GNDD
- J_M4_ENCODER1 pad 2: GNDD -> /M4_ENC_A
- J_M4_ENCODER1 pad 3: /M4_ENC_A -> /M4_ENC_B
- J_M4_ENCODER1 pad 4: /M4_ENC_B -> GNDD
Routing:
- net +5V: track 0.00 -> 306.2 mm, vias 0 -> 3
- net /POWER+: track 0.00 -> 227.4 mm
- net +3.3V: track 0.00 -> 204.2 mm, vias 0 -> 7
- net /MOTORS_STBY: track 0.00 -> 120.4 mm, vias 0 -> 2
- net /M3_ENC_A: track 0.00 -> 101.0 mm
- net /M3_ENC_B: track 0.00 -> 92.6 mm, vias 0 -> 1
- net /LEFT_IN2: track 0.00 -> 92.5 mm, vias 0 -> 1
- net /M2_ENC_B: track 0.00 -> 83.1 mm, vias 0 -> 2
- net /M4_PWM: track 0.00 -> 78.3 mm, vias 0 -> 3
- net /M2_ENC_A: track 0.00 -> 74.2 mm, vias 0 -> 1
- net /ACS_ESP: track 0.00 -> 64.8 mm
- net /M3_PWM: track 0.00 -> 62.7 mm, vias 0 -> 2
- net /M4_ENC_A: track 0.00 -> 57.6 mm
- net /M1_ENC_A_ESP: track 0.00 -> 54.8 mm, vias 0 -> 2
- net /M4_ENC_B: track 0.00 -> 54.5 mm
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- added copper zone on B.Cu, net GNDD
- added copper zone on F.Cu, net GNDD
Other:
- board outline added: 97.1 x 116 mm
