File: ros2/main.kicad_sch (KiCad schematic)
At the start: 17 parts, among them J1 Battery, U1 ESP32-DEVKIT-V1, U2 TB6612NFG, U3 TB6612NFG, U4 ACS712, U5 XL63070, U6 ZC323900, U7 TB6612NFG, U8 TB6612NFG

Commit message: some fix
Parts:
- U6: value ZC323900 -> TXS0108E
Connections:
- net at U7.10 (PWMB): now also U7.16 (PWMA)
- net at U7.11 (BI2): now also U7.15 (AI2)
- net at U7.12 (BI1): now also U7.14 (AI1)
- net at U7.4 (A01): now also U7.7 (B01)
- net at U7.5 (A02): now also U7.6 (B02)
- no-connect marks 95 -> 84
Other:
- note added: "Battery switch"
Changed lines of the file:
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@@
 		)
 	)
+	(text "Battery switch"
+		(exclude_from_sim no)
+		(at 38.862 117.348 0)
+		(effects
+			(font
+				(size 1.27 1.27)
+			)
+		)
+	)
 	(text "5V probably, should be reviewed"
 		(exclude_from_sim no)
@@
 	)
 	(no_connect
-		(at 259.08 55.88)
-	)
-	(no_connect
 		(at 154.94 85.09)
 	)
@@
 	)
 	(no_connect
-		(at 228.6 45.72)
-	)
-	(no_connect
 		(at 73.66 85.09)
 	)
@@
 	)
 	(no_connect
-		(at 228.6 55.88)
-	)
-	(no_connect
 		(at 185.42 48.26)
 	)
@@
 	)
 	(no_connect
-		(at 259.08 45.72)
-	)
-	(no_connect
 		(at 104.14 77.47)
 	)
@@
 	)
 	(no_connect
-		(at 259.08 48.26)
-	)
-	(no_connect
 		(at 147.32 152.4)
 	)
@@
 	)
 	(no_connect
-		(at 259.08 53.34)
-	)
-	(no_connect
 		(at 177.8 139.7)
 	)
 	(no_connect
-		(at 228.6 48.26)
-	)
-	(no_connect
 		(at 104.14 57.15)
 	)
@@
 	)
 	(no_connect
-		(at 228.6 40.64)
-	)
-	(no_connect
 		(at 73.66 69.85)
 	)
@@
 	)
 	(no_connect
-		(at 228.6 38.1)
-	)
-	(no_connect
-		(at 259.08 40.64)
-	)
-	(no_connect
 		(at 154.94 102.87)
 	)
@@
 	)
 	(no_connect
-		(at 228.6 53.34)
-	)
-	(no_connect
 		(at 177.8 132.08)
 	)
@@
 	(wire
 		(pts
+			(xy 227.33 48.26) (xy 227.33 55.88)
+		)
+		(stroke
+			(width 0)
+			(type default)
+		)
+	)
+	(wire
+		(pts
 			(xy 265.43 82.55) (xy 265.43 86.36)
 		)
@@
 	(wire
 		(pts
+			(xy 261.62 53.34) (xy 261.62 45.72)
+		)
+		(stroke
+			(width 0)
+			(type default)
+		)
+	)
+	(wire
+		(pts
+			(xy 226.06 45.72) (xy 226.06 53.34)
+		)
+		(stroke
+			(width 0)
+			(type default)
+		)
+	)
+	(wire
+		(pts
 			(xy 265.43 86.36) (xy 257.81 86.36)
 		)
@@
 	(wire
 		(pts
+			(xy 260.35 48.26) (xy 260.35 55.88)
+		)
+		(stroke
+			(width 0)
+			(type default)
+		)
+	)
+	(wire
+		(pts
 			(xy 185.42 60.96) (xy 185.42 63.5)
 		)
@@
 	(wire
 		(pts
+			(xy 259.08 53.34) (xy 261.62 53.34)
+		)
+		(stroke
+			(width 0)
+			(type default)
+		)
+	)
+	(wire
+		(pts
 			(xy 198.12 38.1) (xy 200.66 38.1)
 		)
@@
 	(wire
 		(pts
+			(xy 228.6 48.26) (xy 227.33 48.26)
+		)
+		(stroke
+			(width 0)
+			(type default)
+		)
+	)
+	(wire
+		(pts
 			(xy 49.53 118.11) (xy 53.34 118.11)
 		)
@@
 	(wire
 		(pts
+			(xy 227.33 55.88) (xy 228.6 55.88)
+		)
+		(stroke
+			(width 0)
+			(type default)
+		)
+	)
+	(wire
+		(pts
 			(xy 68.58 123.19) (xy 77.47 123.19)
 		)
@@
 	(wire
 		(pts
+			(xy 259.08 55.88) (xy 260.35 55.88)
+		)
+		(stroke
+			(width 0)
+			(type default)
+		)
+	)
+	(wire
+		(pts
 			(xy 177.8 157.48) (xy 179.07 157.48)
 		)
@@
 	(wire
 		(pts
+			(xy 226.06 53.34) (xy 228.6 53.34)
+		)
+		(stroke
+			(width 0)
+			(type default)
+		)
+	)
+	(wire
+		(pts
 			(xy 266.7 38.1) (xy 259.08 38.1)
 		)
@@
 	(wire
 		(pts
+			(xy 259.08 45.72) (xy 261.62 45.72)
+		)
+		(stroke
+			(width 0)
+			(type default)
+		)
+	)
+	(wire
+		(pts
+			(xy 228.6 45.72) (xy 226.06 45.72)
+		)
+		(stroke
+			(width 0)
+			(type default)
+		)
+	)
+	(wire
+		(pts
 			(xy 123.19 144.78) (xy 127 144.78)
 		)
@@
 	(wire
 		(pts
-			(xy 45.72 118.11) (xy 49.53 118.11)
+			(xy 259.08 48.26) (xy 260.35 48.26)
+		)
+		(stroke
+			(width 0)
+			(type default)
+		)
+	)
+	(wire
+		(pts
+			(xy 22.86 118.11) (xy 49.53 118.11)
 		)
 		(stroke
@@
 		)
 	)
+	(wire
+		(pts
+			(xy 228.6 38.1) (xy 228.6 40.64)
+		)
+		(stroke
+			(width 0)
+			(type default)
+		)
+	)
 	(label "POWER+"
 		(at 101.6 139.7 180)
@@
 	)
 	(label "POWER+"
-		(at 45.72 118.11 180)
+		(at 24.13 118.11 180)
 		(effects
 			(font
@@
 			)
 		)
-		(property "Value" "ZC323900"
+		(property "Value" "TXS0108E"
 			(at 162.56 116.84 0)
 			(show_name no)

Commit message: schema without esp32
Parts:
- removed C3, C5, C7: 100nF, symbol Device:C_Small
- removed C4, C6, C8: 10uF, symbol Device:C_Small
- removed J1: Battery, Battery:Connector, symbol Connector:Conn_01x02_Socket
- removed U4: ACS712, Package_SO:SOIC-8_3.9x4.9mm_P1.27mm, symbol ACS712:ACS712
- removed U8: TB6612NFG, tb6612fng:MODULE_ROB-14450, symbol ROB-14450:ROB-14450
- added C10, C4, C6, C8: 220uF, symbol Device:C_Polarized
- added C13: 100nF, symbol Device:C_Small
- added C14: 10uF, symbol Device:C_Small
- added C15: 22uF, symbol Device:C
- added C16, C18, C19, C20: 100nF, symbol Device:C
- added C17: 2200uF, symbol Device:C_Polarized
- added C3, C5, C7, C9: 22nF, symbol Device:C
- added D1: LED, symbol Device:LED
- added H1, H2, H3, H4: MountingHole, symbol Mechanical:MountingHole
- added J1: Battery Conn_01x02, TerminalBlock:TerminalBlock_Xinya_XY308-2.54-2P_1x02_P2.54mm_Horizontal, symbol Connector_Generic:Conn_01x02
- added J2: BMS_input, Connector_Wire:SolderWire-1sqmm_1x03_P5.4mm_D1.4mm_OD2.7mm, symbol Connector_Generic:Conn_01x03
- added J3: BMS_output, Connector_Wire:SolderWire-1sqmm_1x02_P5.4mm_D1.4mm_OD2.7mm, symbol Connector_Generic:Conn_01x02
- added J4: Conn_01x03, symbol Connector_Generic:Conn_01x03
- added J5: SWITCH_CONNECTOR, Connector_Wire:SolderWire-1sqmm_1x02_P5.4mm_D1.4mm_OD2.7mm, symbol Connector_Generic:Conn_01x02
- added J_M1_ENCODER1, J_M2_ENCODER1, J_M3_ENCODER1, J_M4_ENCODER1: Conn_01x04, Connector_PinHeader_2.54mm:PinHeader_1x04_P2.54mm_Vertical, symbol Connector_Generic:Conn_01x04
- added J_M1_POWER1, J_M2_POWER1, J_M3_POWER1, J_M4_POWER1: Conn_01x02, TerminalBlock:TerminalBlock_Xinya_XY308-2.54-2P_1x02_P2.54mm_Horizontal, symbol Connector_Generic:Conn_01x02
- added R1: 1k, symbol Device:R
- added R2, R4: 10K, symbol Device:R
- added R3: 100K, symbol Device:R
- added SW1: MRS-101, symbol Switch:SW_SPST
- added U5: TB6612NFG, tb6612fng:MODULE_ROB-14450, symbol ROB-14450:ROB-14450
- added U7: (no value), ACS712_MODULE:ACS712_module, symbol ACS712_Module:ACS712_30A
- renumbered U7 to U4, U5 to U8
Connections:
- net POWER- is gone; now on net GND: U8.2 (GND)
- net +3.3V: now also U2.2 (VCC), U3.2 (VCC), U4.2 (VCC), U6.1 (VA), C19.1, U5.2 (VCC)
- net +5V: now also U1.30 (VIN), U6.20 (VB), C13.1, C14.1, C15.1, C16.1, C18.1, J_M1_ENCODER1.1 (Pin_1), J_M2_ENCODER1.1 (Pin_1), J_M3_ENCODER1.1 (Pin_1), J_M4_ENCODER1.1 (Pin_1), U7.1 (Vcc); no longer U2.2 (VCC), U3.2 (VCC), U4.2 (VCC)
- net GND: now also C10.2, C13.2, C14.2, C15.2, C16.2, C17.2, C18.2, C19.2, C20.2, C3.2, C4.2, C5.2, C6.2, C7.2, C8.2, C9.2, D1.1 (K), J3.2 (Pin_2), J_M1_ENCODER1.2 (Pin_2), J_M2_ENCODER1.2 (Pin_2), J_M3_ENCODER1.2 (Pin_2), J_M4_ENCODER1.2 (Pin_2), R3.2, R4.2, U5.3 (GND), U5.8 (GND), U5.9 (GND), U7.3 (GND)
- net POWER+: now also U2.1 (VM), U3.1 (VM), U4.1 (VM), C10.1, C17.1, C3.1, C4.1, C5.1, C6.1, C7.1, C8.1, C9.1, J5.2 (Pin_2), R1.1, SW1.2 (B), U5.1 (VM)
- net M4_PWM: now reaches U4.10 (PWMB), U4.16 (PWMA)
- net M4_IN2: now reaches U4.11 (BI2), U4.15 (AI2)
- net M4_IN1: now reaches U4.12 (BI1), U4.14 (AI1)
- net MOTORS_STBY: now reaches U4.13 (STBY)
- net MOTORS_STBY: now also U2.13 (STBY), U3.13 (STBY), U5.13 (STBY)
- net M4_OUT1: now reaches U4.4 (A01), U4.7 (B01)
- net M4_OUT1: now also J_M4_POWER1.1 (Pin_1)
- net M4_OUT2: now reaches U4.5 (A02), U4.6 (B02)
- net M4_OUT2: now also J_M4_POWER1.2 (Pin_2)
- net M3_PWM: now reaches U3.10 (PWMB)
- net M3_PWM: now also U3.16 (PWMA)
- net M3_IN2: now reaches U3.11 (BI2)
- net M3_IN2: now also U3.15 (AI2)
- net M3_IN1: now reaches U3.12 (BI1)
- net M3_IN1: now also U3.14 (AI1)
- net M3_OUT1: now reaches U3.4 (A01)
- net M3_OUT1: now also U3.7 (B01), J_M2_POWER1.1 (Pin_1)
- net M3_OUT2: now reaches U3.5 (A02)
- net M3_OUT2: now also U3.6 (B02), J_M2_POWER1.2 (Pin_2)
- net M2_PWM: now reaches U2.10 (PWMB)
- net M2_PWM: now also U2.16 (PWMA)
- net M2_IN2: now reaches U2.11 (BI2)
- net M2_IN2: now also U2.15 (AI2)
- net M2_IN1: now reaches U2.12 (BI1)
- net M2_IN1: now also U2.14 (AI1)
- net M2_OUT1: now reaches U2.4 (A01)
- net M2_OUT1: now also U2.7 (B01), J_M3_POWER1.1 (Pin_1)
- net M2_OUT2: now reaches U2.5 (A02)
- net M2_OUT2: now also U2.6 (B02), J_M3_POWER1.2 (Pin_2)
- net TXS_OE: now reaches U6.10 (OE)
- net TXS_OE: now also R3.1
- net M4_ENC_B: now reaches U6.12 (B8)
- net M4_ENC_B: now also J_M4_ENCODER1.4 (Pin_4)
- net M4_ENC_A: now reaches U6.13 (B7)
- net M4_ENC_A: now also J_M4_ENCODER1.3 (Pin_3)
- net M3_ENC_B: now reaches U6.14 (B6)
- net M3_ENC_B: now also J_M2_ENCODER1.4 (Pin_4)
- net M3_ENC_A: now reaches U6.15 (B5)
- net M3_ENC_A: now also J_M2_ENCODER1.3 (Pin_3)
- net M2_ENC_B: now reaches U6.16 (B4)
- net M2_ENC_B: now also J_M3_ENCODER1.4 (Pin_4)
- net M2_ENC_A: now reaches U6.17 (B3)
- net M2_ENC_A: now also J_M3_ENCODER1.3 (Pin_3)
- net M1_ENC_B: now reaches U6.18 (B2)
- net M1_ENC_B: now also J_M1_ENCODER1.4 (Pin_4)
- net M1_ENC_A: now reaches U6.19 (B1)
- net M1_ENC_A: now also J_M1_ENCODER1.3 (Pin_3)
- net M1_ENC_A_ESP: now reaches U6.2 (A1)
- net M1_ENC_B_ESP: now reaches U6.3 (A2)
- net M2_ENC_A_ESP: now reaches U6.4 (A3)
- net M2_ENC_B_ESP: now reaches U6.5 (A4)
- net M3_ENC_A_ESP: now reaches U6.6 (A5)
- net M3_ENC_B_ESP: now reaches U6.7 (A6)
- net M4_ENC_A_ESP: now reaches U6.8 (A7)
- net M4_ENC_B_ESP: now reaches U6.9 (A8)
- new net: R2.1, U7.2 (OUT)
- new net: D1.2 (A), R1.2
- new net ACS_ESP: C20.1, R2.2, R4.1
- new net BAT_MID: J2.2 (Pin_2), J4.2 (Pin_2)
- new net BAT_RAW_MINUS: J1.2 (Pin_2), J2.3 (Pin_3), J4.3 (Pin_3)
- new net BAT_RAW_PLUS: J1.1 (Pin_1), J2.1 (Pin_1), J4.1 (Pin_1)
- new net BMS P+: J3.1 (Pin_1), J5.1 (Pin_1), SW1.1 (A)
- new net M1_IN1: U5.12 (BI1), U5.14 (AI1)
- new net M1_IN2: U5.11 (BI2), U5.15 (AI2)
- new net M1_OUT1: J_M1_POWER1.1 (Pin_1), U5.4 (A01), U5.7 (B01)
- new net M1_OUT2: J_M1_POWER1.2 (Pin_2), U5.5 (A02), U5.6 (B02)
- new net M1_PWM: U5.10 (PWMB), U5.16 (PWMA)
- no-connect marks 84 -> 26
Other:
- note added: "ACS712_MODULE"
- note added: "BMS 2S"
- note added: "Battery"
- note added: "SWITCH BUTTON"
- note added: "ОДИН З ЦИХ ТРЕБА ЗАБРАТИ"
- note added: "від 510 до 1500 Ом я не визначив нормально"
- note removed: "5V probably, should be reviewed"
- note removed: "Analog output signal, connect to esp32"
- note removed: "Battery switch"
- note removed: "Raw input of battaries"
- moved on the sheet: C1, C2, U1, U4, U6, U8

Commit message: add esp32 connections
Parts:
- added C21: 100nF, Capacitor_THT:C_Disc_D5.0mm_W2.5mm_P5.00mm, symbol Device:C
- added J6: ACS_IN, Connector_Wire:SolderWire-1sqmm_1x01_D1.4mm_OD2.7mm, symbol Connector_Generic:Conn_01x01
- added J7: ACS_POWER_OUT, Connector_Wire:SolderWire-1sqmm_1x01_D1.4mm_OD2.7mm, symbol Connector_Generic:Conn_01x01
- added R5: 30К, Resistor_THT:R_Axial_DIN0207_L6.3mm_D2.5mm_P7.62mm_Horizontal, symbol Device:R
- added R6: 10K, Resistor_THT:R_Axial_DIN0207_L6.3mm_D2.5mm_P7.62mm_Horizontal, symbol Device:R
- C1, C13, C14, C15, C16, C18, C19, C2, C20, C3, C5, C7, C9: footprint (none) -> Capacitor_THT:C_Disc_D5.0mm_W2.5mm_P5.00mm
- C10, C4, C6, C8: footprint (none) -> Capacitor_THT:CP_Radial_D10.0mm_P3.50mm
- C17: footprint (none) -> Capacitor_THT:CP_Radial_D12.5mm_P5.00mm
- D1: footprint (none) -> LED_THT:LED_D5.0mm
- H1, H2, H3, H4: footprint (none) -> MountingHole:MountingHole_3.2mm_M3
- J5: value SWITCH_CONNECTOR -> SW_CONNECTOR
- R1, R3, R4: footprint (none) -> Resistor_THT:R_Axial_DIN0207_L6.3mm_D2.5mm_P7.62mm_Horizontal
- R2: value 10K -> 10К; footprint (none) -> Resistor_THT:R_Axial_DIN0207_L6.3mm_D2.5mm_P7.62mm_Horizontal
- U7: value (none) -> ACS712_MODULE
Connections:
- net M1_IN1 is gone; now on net LEFT_IN1: U5.12 (BI1), U5.14 (AI1)
- net M1_IN2 is gone; now on net LEFT_IN2: U5.11 (BI2), U5.15 (AI2)
- net M2_IN1 is gone; now on net LEFT_IN1: U2.12 (BI1), U2.14 (AI1)
- net M2_IN2 is gone; now on net LEFT_IN2: U2.11 (BI2), U2.15 (AI2)
- net M3_IN1 is gone; now on net RIGHT_IN1: U3.12 (BI1), U3.14 (AI1)
- net M3_IN2 is gone; now on net RIGHT_IN2: U3.11 (BI2), U3.15 (AI2)
- net M4_IN1 is gone; now on net RIGHT_IN1: U4.12 (BI1), U4.14 (AI1)
- net M4_IN2 is gone; now on net RIGHT_IN2: U4.11 (BI2), U4.15 (AI2)
- net ACS_ESP: now also U1.18 (VN)
- net GND: now also C21.2, R6.2
- net M1_ENC_A_ESP: now also U1.19 (D34)
- net M1_ENC_B_ESP: now also U1.20 (D35)
- net M1_PWM: now also U1.9 (D18)
- net M2_ENC_A_ESP: now also U1.21 (D32)
- net M2_ENC_B_ESP: now also U1.22 (D33)
- net M2_PWM: now also U1.10 (D19)
- net M3_ENC_A_ESP: now also U1.26 (D14)
- net M3_ENC_B_ESP: now also U1.6 (RX2)
- net M3_PWM: now also U1.11 (D21)
- net M4_ENC_A_ESP: now also U1.7 (TX2)
- net M4_ENC_B_ESP: now also U1.5 (D4)
- net M4_PWM: now also U1.14 (D22)
- net MOTORS_STBY: now also U1.28 (D13)
- net POWER+: now also J7.1 (Pin_1), R5.1; no longer J5.2 (Pin_2), SW1.2 (B)
- net TXS_OE: now also U1.4 (D2)
- net LEFT_IN1: now reaches U1.15 (D23)
- net VBAT_ADC: now reaches U1.17 (VP)
- net VBAT_ADC: now also C21.1, R5.2, R6.1
- net LEFT_IN2: now reaches U1.23 (D25)
- net RIGHT_IN1: now reaches U1.24 (D26)
- net RIGHT_IN2: now reaches U1.25 (D27)
- new net SWITCHED_PLUS: J5.2 (Pin_2), J6.1 (Pin_1), SW1.2 (B)
- no-connect marks 26 -> 6
Other:
- note added: "вимірювання напруги батареї"
- note removed: "Review option of making 5V supply so no need in second buck"
- moved on the sheet: C1, C13, C14, C2, C20, D1, J1, J2, J3, J4, J5, R1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

Commit message: comlete schematic no real errors
Parts:
- U1: footprint esp32:MODULE_ESP32_DEVKIT_V1 -> ESP32-DEVKIT-V1:MODULE_ESP32_DEVKIT_V1
- U7: footprint ACS712_MODULE:ACS712_module -> Connector_PinSocket_2.54mm:PinSocket_1x03_P2.54mm_Vertical
Other:
- moved on the sheet: C1, C2, U1

Commit message: saved details
Changed lines of the file:
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@@
 	(text "ОДИН З ЦИХ ТРЕБА ЗАБРАТИ"
 		(exclude_from_sim no)
-		(at 40.64 38.1 0)
+		(at 40.386 38.608 0)
 		(effects
 			(font

Commit message: prettier fix
Other:
- note added: "Buck"
- note added: "LEFT WHEELS"
- note added: "Level shifter"
- note added: "RIGHT WHEELS"
- moved on the sheet: C1, C15, C16, C18, C19, C2, C5, C6, C7, C8, J_M1_ENCODER1, J_M1_POWER1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

Commit message: fix 2
Parts:
- added C11: 100nF, Capacitor_THT:C_Disc_D5.0mm_W2.5mm_P5.00mm, symbol Device:C_Small
- added C12: 10uF, Capacitor_THT:C_Disc_D5.0mm_W2.5mm_P5.00mm, symbol Device:C_Small
- D1: value LED -> LED_RED
Connections:
- net +5V: now also C11.1, C12.1
- net GND: now also C11.2, C12.2

Commit message: routed pcb + corrected schematic
Parts:
- removed J1: Battery Conn_01x02, TerminalBlock:TerminalBlock_Xinya_XY308-2.54-2P_1x02_P2.54mm_Horizontal, symbol Connector_Generic:Conn_01x02
- removed SW1: MRS-101, symbol Switch:SW_SPST
- C3, C5, C7, C9: value 22nF -> 100nF
- J4: footprint (none) -> Connector_Wire:SolderWire-1sqmm_1x03_P5.4mm_D1.4mm_OD2.7mm
- U1: footprint ESP32-DEVKIT-V1:MODULE_ESP32_DEVKIT_V1 -> esp32:MODULE_ESP32_DEVKIT_V1
- U2, U3, U4, U5: footprint tb6612fng:MODULE_ROB-14450 -> ROB-14450:MODULE_ROB-14450
- U7: footprint Connector_PinSocket_2.54mm:PinSocket_1x03_P2.54mm_Vertical -> ACS712_MODULE:ACS712_module
Connections:
- net BAT_RAW_MINUS is gone; now on net GND: J2.3 (Pin_3), J4.3 (Pin_3)
- net GND: now also J_M1_ENCODER1.4 (Pin_4), J_M2_ENCODER1.4 (Pin_4), J_M3_ENCODER1.4 (Pin_4), J_M4_ENCODER1.4 (Pin_4); no longer J_M1_ENCODER1.2 (Pin_2), J_M2_ENCODER1.2 (Pin_2), J_M3_ENCODER1.2 (Pin_2), J_M4_ENCODER1.2 (Pin_2)
- net M1_ENC_A: now also J_M1_ENCODER1.2 (Pin_2); no longer J_M1_ENCODER1.3 (Pin_3)
- net M1_ENC_B: now also J_M1_ENCODER1.3 (Pin_3); no longer J_M1_ENCODER1.4 (Pin_4)
- net M2_ENC_A: now also J_M3_ENCODER1.2 (Pin_2); no longer J_M3_ENCODER1.3 (Pin_3)
- net M2_ENC_B: now also J_M3_ENCODER1.3 (Pin_3); no longer J_M3_ENCODER1.4 (Pin_4)
- net M3_ENC_A: now also J_M2_ENCODER1.2 (Pin_2); no longer J_M2_ENCODER1.3 (Pin_3)
- net M3_ENC_B: now also J_M2_ENCODER1.3 (Pin_3); no longer J_M2_ENCODER1.4 (Pin_4)
- net M4_ENC_A: now also J_M4_ENCODER1.2 (Pin_2); no longer J_M4_ENCODER1.3 (Pin_3)
- net M4_ENC_B: now also J_M4_ENCODER1.3 (Pin_3); no longer J_M4_ENCODER1.4 (Pin_4)
Other:
- note removed: "ОДИН З ЦИХ ТРЕБА ЗАБРАТИ"
- moved on the sheet: C1, C13, C14, C15, C16, C18, C19, C2, C21, C3, C4, C5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
